Commit message: Update mesh file path

File: wx250s/wx250s.urdf (robot description, URDF)
Before this commit: robot wx250s, 14 links, 13 joints
Links:
- removed link wx250s/base_link
- added link base_link, mass 0.538736; collision mesh filename=file://${mesh_dir}/base.stl scale=0.001 0.001 0.001; visual mesh filename=file://${mesh_dir}/base.stl scale=0.001 0.001 0.001
- link wx250s/gripper_bar_link: geometry collision mesh filename=file://${mesh_dir}/gripper_bar.stl scale=0.001 0.001 0.001; visual mesh filename=file://${mesh_dir}/gripper_bar.stl scale=0.001 0.001 0.001
- link wx250s/gripper_link: geometry collision mesh filename=file://${mesh_dir}/gripper.stl scale=0.001 0.001 0.001; visual mesh filename=file://${mesh_dir}/gripper.stl scale=0.001 0.001 0.001
- link wx250s/gripper_prop_link: geometry collision mesh filename=file://${mesh_dir}/gripper_prop.stl scale=0.001 0.001 0.001; visual mesh filename=file://${mesh_dir}/gripper_prop.stl scale=0.001 0.001 0.001
- link wx250s/left_finger_link: geometry collision mesh filename=file://${mesh_dir}/gripper_finger.stl scale=0.001 0.001 0.001; visual mesh filename=file://${mesh_dir}/gripper_finger.stl scale=0.001 0.001 0.001
- link wx250s/lower_forearm_link: geometry collision mesh filename=file://${mesh_dir}/lower_forearm.stl scale=0.001 0.001 0.001; visual mesh filename=file://${mesh_dir}/lower_forearm.stl scale=0.001 0.001 0.001
- link wx250s/right_finger_link: geometry collision mesh filename=file://${mesh_dir}/gripper_finger.stl scale=0.001 0.001 0.001; visual mesh filename=file://${mesh_dir}/gripper_finger.stl scale=0.001 0.001 0.001
- link wx250s/shoulder_link: geometry collision mesh filename=file://${mesh_dir}/shoulder.stl scale=0.001 0.001 0.001; visual mesh filename=file://${mesh_dir}/shoulder.stl scale=0.001 0.001 0.001
- link wx250s/upper_arm_link: geometry collision mesh filename=file://${mesh_dir}/upper_arm.stl scale=0.001 0.001 0.001; visual mesh filename=file://${mesh_dir}/upper_arm.stl scale=0.001 0.001 0.001
- link wx250s/upper_forearm_link: geometry collision mesh filename=file://${mesh_dir}/upper_forearm.stl scale=0.001 0.001 0.001; visual mesh filename=file://${mesh_dir}/upper_forearm.stl scale=0.001 0.001 0.001
- link wx250s/wrist_link: geometry collision mesh filename=file://${mesh_dir}/wrist.stl scale=0.001 0.001 0.001; visual mesh filename=file://${mesh_dir}/wrist.stl scale=0.001 0.001 0.001
Joints:
- joint waist: parent wx250s/base_link -> base_link
